Commit message: Update snake_bot.urdf

File: snake_bot.urdf (robot description, URDF)
Before this commit: robot snake_bot, 7 links, 6 joints
Links:
- link base_link: mass None -> 1.0; geometry collision cylinder length=0.07 radius=0.03; visual cylinder length=0.07 radius=0.03
- link link1: mass None -> 0.5; geometry collision cylinder length=0.07 radius=0.03; visual cylinder length=0.07 radius=0.03
- link link2: mass None -> 0.5; geometry collision cylinder length=0.07 radius=0.03; visual cylinder length=0.07 radius=0.03
- link link3: mass None -> 0.5; geometry collision cylinder length=0.07 radius=0.03; visual cylinder length=0.07 radius=0.03
- link link4: mass None -> 0.5; geometry collision cylinder length=0.07 radius=0.03; visual cylinder length=0.07 radius=0.03
- link link5: mass None -> 0.5; geometry collision cylinder length=0.07 radius=0.03; visual cylinder length=0.07 radius=0.03
- link link6: mass None -> 0.5; geometry collision cylinder length=0.07 radius=0.03; visual cylinder length=0.07 radius=0.03
